File: PCBs/remote_board/shark_bait_remote.kicad_pcb (KiCad board)
At the start: 2 copper layers, 110 x 75 mm, 41 parts, among them J1 BATT+, J10 PRIME, J11 ARM, J12 GPSLED, J13 PLED, J14 ARMLED, J15 Conn_01x06, J2 BATT-, J3 15MIN, J4 12H, J5 MTRDIR, J6 FLOW, J7 SERVO, J8 MOTOR+, J9 MOTOR-, Q1 MMBT3904, U1 CD74HC4067M, U2 TSR_1-2450, U3 CD74HC4067M

Commit message: updated PCBs and Ordered
Parts:
- removed G***: LOGO, logos:SH_Logo
- removed G***: LOGO, logos:SH_Logo_cu
- removed G***: LOGO, logos:shark_bait_logo
- removed JP3: PinHeader_01x12_2.54mm, Adafruit_FeatherWing:Conn_PinHeader_1x12_Reduced
- removed JP4: PinHeader_01x16_2.54mm, Adafruit_FeatherWing:Conn_PinHeader_1x16_Reduced
- removed the PCB** at (160.9, 73.7)
- removed the PCB** at (137.1, 73.7)
- removed the PCB** at (112.9, 73.7)
- added C5: 0.1uF, Capacitor_SMD:C_0805_2012Metric, F.Cu at (124.0, 49.5)
- added C6: 0.1uF, Capacitor_SMD:C_0805_2012Metric, F.Cu at (199.0, 50.0)
- added C7: 0.1uF, Capacitor_SMD:C_0805_2012Metric, F.Cu at (175.0, 50.0)
- added C8: 0.1uF, Capacitor_SMD:C_0805_2012Metric, F.Cu at (149.5, 50.0)
- added PCB**: VAL**, Adafruit_FeatherWing:PCB_FeatherWing_NoHoles, F.Cu at (152.0, 68.0)
- added Q2: MMBT3904, Package_TO_SOT_SMD:SOT-23, F.Cu at (130.5, 87.5)
- added Q3: MMBT3904, Package_TO_SOT_SMD:SOT-23, F.Cu at (137.5, 87.5)
- added Q4: MMBT3904, Package_TO_SOT_SMD:SOT-23, F.Cu at (151.5, 87.5)
- added Q5: MMBT3904, Package_TO_SOT_SMD:SOT-23, F.Cu at (158.5, 87.5)
- added Q6: MMBT3904, Package_TO_SOT_SMD:SOT-23, F.Cu at (165.5, 87.5)
- added Q7: MMBT3904, Package_TO_SOT_SMD:SOT-23, F.Cu at (172.5, 87.5)
- added Q8: MMBT3904, Package_TO_SOT_SMD:SOT-23, F.Cu at (179.5, 87.5)
- added R10: 1k, Resistor_SMD:R_0805_2012Metric, F.Cu at (130.5, 84.5)
- added R11: 1k, Resistor_SMD:R_0805_2012Metric, F.Cu at (137.5, 84.5)
- added R12: 1k, Resistor_SMD:R_0805_2012Metric, F.Cu at (151.5, 84.5)
- added R13: 1k, Resistor_SMD:R_0805_2012Metric, F.Cu at (155.5, 88.5)
- added R14: 1k, Resistor_SMD:R_0805_2012Metric, F.Cu at (162.5, 88.4)
- added R15: 1k, Resistor_SMD:R_0805_2012Metric, F.Cu at (169.5, 88.5)
- added R16: 1k, Resistor_SMD:R_0805_2012Metric, F.Cu at (176.5, 88.5)
- added R17: 1k, Resistor_SMD:R_0805_2012Metric, F.Cu at (158.5, 84.5)
- added R18: 1k, Resistor_SMD:R_0805_2012Metric, F.Cu at (165.5, 84.5)
- added R19: 1k, Resistor_SMD:R_0805_2012Metric, F.Cu at (172.5, 84.5)
- added R20: 1k, Resistor_SMD:R_0805_2012Metric, F.Cu at (179.6, 84.5)
- added R21: 10K, Resistor_SMD:R_0805_2012Metric, F.Cu at (107.5, 87.5)
- added R22: 10K, Resistor_SMD:R_0805_2012Metric, F.Cu at (114.5, 87.5)
- added R7: 1k, Resistor_SMD:R_0805_2012Metric, F.Cu at (134.5, 88.5)
- added R8: 1k, Resistor_SMD:R_0805_2012Metric, F.Cu at (141.5, 88.5)
- added R9: 1k, Resistor_SMD:R_0805_2012Metric, F.Cu at (148.5, 88.5)
- added SW1: PUSH, Connector_JST:JST_PH_B2B-PH-K_1x02_P2.00mm_Vertical, F.Cu at (106.5, 93.0)
- added SW2: PUSH, Connector_JST:JST_PH_B2B-PH-K_1x02_P2.00mm_Vertical, F.Cu at (113.5, 93.0)
- added U4: CD74HC4067M, Package_SO:SOIC-24W_7.5x15.4mm_P1.27mm, F.Cu at (164.0, 46.0)
- added U5: CD74HC4067M, Package_SO:SOIC-24W_7.5x15.4mm_P1.27mm, F.Cu at (114.0, 46.0)
- J10: value PRIME -> LED
- J11: value ARM -> LED
- J12: value GPSLED -> LED
- J14: value ARMLED -> LED
- J15: value Conn_01x06 -> LED; footprint project_footprints:Nidec_CS-7 -> Connector_JST:JST_PH_B2B-PH-K_1x02_P2.00mm_Vertical
- J3: value 15MIN -> FLOW1; footprint Connector_JST:JST_PH_B5B-PH-K_1x05_P2.00mm_Vertical -> Connector_JST:JST_PH_B11B-PH-K_1x11_P2.00mm_Vertical
- J4: value 12H -> FLOW1; footprint Connector_JST:JST_PH_B13B-PH-K_1x13_P2.00mm_Vertical -> Connector_JST:JST_PH_B11B-PH-K_1x11_P2.00mm_Vertical
- J5: value MTRDIR -> FLOW1; footprint Connector_JST:JST_PH_B2B-PH-K_1x02_P2.00mm_Vertical -> Connector_JST:JST_PH_B11B-PH-K_1x11_P2.00mm_Vertical
- J6: value FLOW -> FLOW1
- J7: value SERVO -> LED; footprint Connector_JST:JST_PH_B3B-PH-K_1x03_P2.00mm_Vertical -> Connector_JST:JST_PH_B2B-PH-K_1x02_P2.00mm_Vertical
- J8: value MOTOR+ -> LED; footprint project_footprints:connect_QC_Male -> Connector_JST:JST_PH_B2B-PH-K_1x02_P2.00mm_Vertical
- J9: value MOTOR- -> LED; footprint project_footprints:connect_QC_Male -> Connector_JST:JST_PH_B2B-PH-K_1x02_P2.00mm_Vertical
- R5: value 330 -> 1k
- moved J7 83.0 mm to (129.0, 93.0)
- moved J5 72.2 mm to (104.0, 35.0)
- moved J8 71.5 mm to (136.0, 93.0)
- moved J11 68.9 mm to (164.0, 93.0)
- moved J10 66.9 mm to (157.0, 93.0)
- moved J15 62.1 mm to (178.0, 93.0), turned to 0 degrees
- moved R5 58.0 mm to (127.5, 88.5), turned to 90 degrees
- moved J9 54.5 mm to (150.0, 93.0)
- moved JP1 52.7 mm to (152.1, 55.0), turned to 0 degrees
- moved C4 47.2 mm to (126.0, 49.5), turned to 270 degrees
- moved C2 45.3 mm to (177.0, 50.0), turned to 270 degrees
- moved J4 45.3 mm to (154.0, 35.0)
- moved R4 44.5 mm to (128.0, 49.5)
- moved J14 40.1 mm to (143.0, 93.0), turned to 0 degrees
- moved Q1 37.3 mm to (144.5, 87.5), turned to 270 degrees
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Connections:
- net /SCL renamed LED2
- net /SDA renamed LED1
- J10 pad 1: PRIME -> Net-(J10-Pad1)
- J10 pad 2: GND -> Net-(J10-Pad2)
- J11 pad 1: ARM -> Net-(J11-Pad1)
- J11 pad 2: GND -> Net-(J11-Pad2)
- J12 pad 2: GND -> Net-(J12-Pad2)
- J14 pad 1: +BATT -> Net-(J14-Pad1)
- J15 pad 2: GND -> Net-(J15-Pad2)
- J3 pad 5: GND -> Net-(J3-Pad5)
- J4 pad 11: Net-(J4-Pad11) -> GND
- J5 pad 2: GND -> Net-(J5-Pad2)
- J7 pad 1: +5V -> Net-(J7-Pad1)
- J7 pad 2: Servo -> Net-(J7-Pad2)
- J8 pad 1: +BATT -> Net-(J8-Pad1)
- J9 pad 1: GND -> Net-(J9-Pad1)
- JP1 pad 10: /A2 -> S2
- JP1 pad 11: PRIME -> S1
- JP1 pad 12: ARM -> S0
- JP1 pad 2: /D1 -> KNOB4
- JP1 pad 3: /D0 -> KNOB3
- JP1 pad 7: /A5 -> KNOB2
- JP1 pad 8: /A4 -> KNOB1
- JP1 pad 9: /A3 -> S3
- JP2 pad 3: Servo -> LED3
- JP2 pad 4: /D6 -> LED4
- JP2 pad 5: ARMLED -> BUTT1
- JP2 pad 6: GPSLED -> LED5
- JP2 pad 7: /D11 -> LED6
- JP2 pad 8: /D12 -> LED7
- JP2 pad 9: /D13 -> LED8
- JP5 pad 3: Servo -> LED3
- JP5 pad 4: /D6 -> LED4
- JP5 pad 5: ARMLED -> BUTT1
- JP5 pad 6: GPSLED -> LED5
- JP5 pad 7: /D11 -> LED6
- JP5 pad 8: /D12 -> LED7
- JP5 pad 9: /D13 -> LED8
- JP6 pad 10: /A2 -> S2
- JP6 pad 11: PRIME -> S1
- JP6 pad 12: ARM -> S0
- JP6 pad 2: /D1 -> KNOB4
- JP6 pad 3: /D0 -> KNOB3
- JP6 pad 7: /A5 -> KNOB2
- JP6 pad 8: /A4 -> KNOB1
- JP6 pad 9: /A3 -> S3
- R1 pad 2: /D13 -> KNOB3
- R2 pad 2: /D6 -> KNOB1
- R3 pad 2: PRIME -> KNOB2
- R4 pad 2: ARM -> KNOB4
- R5 pad 1: Net-(J12-Pad1) -> Net-(J7-Pad1)
- R5 pad 2: GPSLED -> +5V
- R6 pad 2: ARMLED -> LED3
- U1 pad 1: /D13 -> KNOB3
- U1 pad 10: /MISO -> S0
- U1 pad 11: /MOSI -> S1
- U1 pad 13: /D11 -> S3
- U1 pad 14: /D12 -> S2
- U1 pad 16: Net-(J3-Pad1) -> Net-(U1-Pad16)
- U1 pad 17: Net-(J3-Pad2) -> Net-(U1-Pad17)
- U1 pad 18: Net-(J3-Pad3) -> Net-(U1-Pad18)
- U1 pad 19: Net-(J3-Pad4) -> Net-(U1-Pad19)
- U1 pad 2: Net-(J4-Pad8) -> Net-(J3-Pad8)
- U1 pad 20: Net-(J4-Pad12) -> Net-(U1-Pad20)
- U1 pad 21: Net-(J4-Pad11) -> Net-(U1-Pad21)
- U1 pad 22: Net-(J4-Pad10) -> Net-(J3-Pad10)
- U1 pad 23: Net-(J4-Pad9) -> Net-(J3-Pad9)
- U1 pad 3: Net-(J4-Pad7) -> Net-(J3-Pad7)
- U1 pad 4: Net-(J4-Pad6) -> Net-(J3-Pad6)
- U1 pad 5: Net-(J4-Pad5) -> Net-(J3-Pad5)
- U1 pad 6: Net-(J4-Pad4) -> Net-(J3-Pad4)
- U1 pad 7: Net-(J4-Pad3) -> Net-(J3-Pad3)
- U1 pad 8: Net-(J4-Pad2) -> Net-(J3-Pad2)
- U1 pad 9: Net-(J4-Pad1) -> Net-(J3-Pad1)
- U3 pad 1: /D6 -> KNOB1
- U3 pad 10: /A3 -> S0
- U3 pad 11: /A2 -> S1
- U3 pad 13: /A4 -> S3
- U3 pad 14: /A5 -> S2
- U3 pad 17: Net-(J15-Pad6) -> Net-(U3-Pad17)
- U3 pad 18: Net-(J15-Pad4) -> Net-(U3-Pad18)
- U3 pad 19: Net-(J15-Pad3) -> Net-(U3-Pad19)
- U3 pad 20: Net-(J15-Pad1) -> Net-(U3-Pad20)
- U3 pad 21: Net-(J5-Pad1) -> Net-(U3-Pad21)
Routing:
- net PRIME: track 131.1 -> 0.00 mm, vias 1 -> 0
- net ARM: track 120.6 -> 0.00 mm, vias 1 -> 0
- net Servo: track 113.5 -> 0.00 mm
- net /D6: track 104.2 -> 0.00 mm
- net S0: track 0.00 -> 103.4 mm, vias 0 -> 5
- net S1: track 0.00 -> 102.3 mm, vias 0 -> 5
- net /MISO: track 104.5 -> 3.00 mm
- net /D13: track 100.2 -> 0.00 mm
- net /MOSI: track 101.5 -> 3.00 mm
- net S3: track 0.00 -> 97.7 mm, vias 0 -> 5
- net S2: track 0.00 -> 94.1 mm, vias 0 -> 4
- net +5V: track 201.2 -> 109.5 mm
- net /A3: track 88.5 -> 0.00 mm
- net /D11: track 85.6 -> 0.00 mm
- net /A2: track 85.5 -> 0.00 mm
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