File: PCBs/remote_board/shark_bait_remote.sch (KiCad schematic (older format))
At the start: 25 parts, among them J1 BATT+, J10 PRIME, J11 ARM, J13 PLED, J14 ARMLED, J2 BATT-, J6 FLOW1, J7 SERVO, J8 MOTOR+, J9 MOTOR-, Q1 MMBT3904, U2 TSR_1-2450, U3 CD74HC4067M

Commit message: updated PCBs and Ordered
Parts:
- removed J10: PRIME, Connector_JST:JST_PH_B2B-PH-K_1x02_P2.00mm_Vertical, symbol AP2112k:Conn_01x02
- removed J11: ARM, Connector_JST:JST_PH_B2B-PH-K_1x02_P2.00mm_Vertical, symbol AP2112k:Conn_01x02
- removed J7: SERVO, Connector_JST:JST_PH_B3B-PH-K_1x03_P2.00mm_Vertical, symbol Connector_Generic:Conn_01x03
- removed J8: MOTOR+, project_footprints:connect_QC_Male, symbol Connector_Generic:Conn_01x01
- removed J9: MOTOR-, project_footprints:connect_QC_Male, symbol Connector_Generic:Conn_01x01
- removed JP1, JP4: PinHeader_01x16_2.54mm, Adafruit_FeatherWing:Conn_PinHeader_1x16_Reduced, symbol Connector_Generic:Conn_01x16
- removed JP2, JP3: PinHeader_01x12_2.54mm, Adafruit_FeatherWing:Conn_PinHeader_1x12_Reduced, symbol Connector_Generic:Conn_01x12
- removed R3, R4: 10K, Resistor_SMD:R_0805_2012Metric, symbol Device:R_Small
- added C1, C2, C5, C6, C7, C8: 0.1uF, Capacitor_SMD:C_0805_2012Metric, symbol shark_bait_remote-rescue:AP2112k_C_Small-shark_bait_remote-rescue
- added J10, J11, J12, J15, J7, J8, J9: LED, Connector_JST:JST_PH_B2B-PH-K_1x02_P2.00mm_Vertical, symbol shark_bait_remote-rescue:AP2112k_Conn_01x02-shark_bait_remote-rescue
- added J3, J4, J5: FLOW1, Connector_JST:JST_PH_B11B-PH-K_1x11_P2.00mm_Vertical, symbol shark_bait_remote-rescue:Connector_Generic_Conn_01x11-shark_bait_remote-rescue
- added JP1: PinHeader_01x16_2.54mm, Adafruit_FeatherWing:Conn_PinHeader_1x16_Reduced, symbol shark_bait_remote-rescue:Connector_Generic_Conn_01x16-shark_bait_remote-rescue
- added JP2: PinHeader_01x12_2.54mm, Adafruit_FeatherWing:Conn_PinHeader_1x12_Reduced, symbol shark_bait_remote-rescue:Connector_Generic_Conn_01x12-shark_bait_remote-rescue
- added Q2, Q3, Q4, Q5, Q6, Q7, Q8: MMBT3904, Package_TO_SOT_SMD:SOT-23, symbol shark_bait_remote-rescue:Transistor_BJT_MMBT3904-shark_bait_remote-rescue
- added R1, R21, R22, R3, R4: 10K, Resistor_SMD:R_0805_2012Metric, symbol shark_bait_remote-rescue:Device_R_Small-shark_bait_remote-rescue
- added R10, R11, R12, R13, R14, R15, R16, R17, R18, R19, R20, R5, R7, R8, R9: 1k, Resistor_SMD:R_0805_2012Metric, symbol shark_bait_remote-rescue:Device_R_Small-shark_bait_remote-rescue
- added SW1, SW2: PUSH, Connector_JST:JST_PH_B2B-PH-K_1x02_P2.00mm_Vertical, symbol shark_bait_remote-rescue:SW_PUSH_SMALL_H-shark_bait_remote-rescue
- added U1, U4, U5: CD74HC4067M, Package_SO:SOIC-24W_7.5x15.4mm_P1.27mm, symbol shark_bait_remote-rescue:74xx_CD74HC4067M-shark_bait_remote-rescue
- C3, C4: symbol AP2112k:C_Small -> shark_bait_remote-rescue:AP2112k_C_Small-shark_bait_remote-rescue
- J1, J2: symbol Connector_Generic:Conn_01x01 -> shark_bait_remote-rescue:Connector_Generic_Conn_01x01-shark_bait_remote-rescue
- J13: symbol AP2112k:Conn_01x02 -> shark_bait_remote-rescue:AP2112k_Conn_01x02-shark_bait_remote-rescue
- J14: value ARMLED -> LED; symbol AP2112k:Conn_01x02 -> shark_bait_remote-rescue:AP2112k_Conn_01x02-shark_bait_remote-rescue
- J6: symbol Connector_Generic:Conn_01x11 -> shark_bait_remote-rescue:Connector_Generic_Conn_01x11-shark_bait_remote-rescue
- JP5: symbol Connector_Generic:Conn_01x12 -> shark_bait_remote-rescue:Connector_Generic_Conn_01x12-shark_bait_remote-rescue
- JP6: symbol Connector_Generic:Conn_01x16 -> shark_bait_remote-rescue:Connector_Generic_Conn_01x16-shark_bait_remote-rescue
- Q1: symbol Transistor_BJT:MMBT3904 -> shark_bait_remote-rescue:Transistor_BJT_MMBT3904-shark_bait_remote-rescue
- R2, R6: symbol Device:R_Small -> shark_bait_remote-rescue:Device_R_Small-shark_bait_remote-rescue
- U2: symbol Regulator_Switching:TSR_1-2450 -> shark_bait_remote-rescue:Regulator_Switching_TSR_1-2450-shark_bait_remote-rescue
- U3: symbol 74xx:CD74HC4067M -> shark_bait_remote-rescue:74xx_CD74HC4067M-shark_bait_remote-rescue
Connections:
- net labels added: BUTT1, KNOB1, KNOB2, KNOB3, KNOB4, LED1, LED2, LED3, LED4, LED5, LED6, LED7, LED8, S0, S1, S2, S3
- net labels removed: A0, A1, A2, A3, A4, A5, ARM, ARMLED, D0, D1, D10, D11, D12, D13, D5, D6, D9, PRIME, SCL, SDA, Servo
- wire segments 97 -> 193
Other:
- moved on the sheet: Q1
